Commit message: made wheel joints and links a macro

File: description/robot.gazebo.xacro (robot description, xacro)
@@ -116,4 +116,6 @@
             <right_joint>rear_right_wheel_joint</right_joint>
             <wheel_separation>${chassis_width}</wheel_separation>
+            <wheel_separation>${chassis_width}</wheel_separation>
+            <wheel_diameter>${wheel_radius * 2}</wheel_diameter>
             <wheel_diameter>${wheel_radius * 2}</wheel_diameter>
             <!-- Limits -->

File: description/robot.include.xacro (robot description, xacro)
@@ -30,4 +30,39 @@
         </inertial>
     </xacro:macro>
+    <xacro:macro name="wheel_joint" params="name parent child xyz side">
+      <joint name="${name}" type="continuous">
+        <parent link="${parent}" />
+        <child link="${child}" />
+        <xacro:if value="${side == 'left'}">
+            <origin xyz="${xyz}" rpy="-${pi/2} 0 0"/>
+            <axis xyz="0 0 1"/>
+        </xacro:if>
+        <xacro:if value="${side == 'right'}">
+            <origin xyz="${xyz}" rpy="${pi/2} 0 0"/>
+            <axis xyz="0 0 -1"/>
+        </xacro:if>
+        <dynamics damping="10.0" friction="10.0"/>
+      </joint>
+    </xacro:macro>
+    <!--<joint_properties damping="1.0" friction="1.0"/> -->
+    <xacro:macro name="wheel_link" params="name in_radius in_length in_mass">
+        <link name="${name}">
+            <visual>
+                <geometry> <!-- the weheels are 60mm diameter, 25mm thick. -->
+                    <cylinder radius="${in_radius}" length="${in_length}"/>
+                </geometry>
+                <material name="black"/>
+            </visual>
+            <collision>
+                <origin xyz="0 0 0" rpy="0 0 0"/>
+                <geometry>
+                    <cylinder length="${in_length}" radius="${in_radius}" />
+                </geometry>
+            </collision>
+            <xacro:inertial_cylinder mass="${in_mass}" length="${in_length}" radius="${in_radius}">
+                <origin xyz="0 0 0" rpy="0 0 0"/>
+            </xacro:inertial_cylinder>
+        </link>
+    </xacro:macro>
     <!-- materials -->
     <material name="white">

File: description/robot.wheels.xacro (robot description, xacro)
@@ -4,100 +4,60 @@
 	<xacro:property name="wheel_length" value="0.03" />
     <xacro:property name="wheel_radius" value="0.025" />
+    <xacro:property name="wheel_mass" value="1.0"/>
 	<!-- front left wheel -->
-	<joint name="front_left_wheel_joint" type = "continuous">
-		<parent link="base_link"/>
-		<child link="front_left_wheel_link"/>
-		<origin xyz="${chassis_length/4} ${chassis_length/2 + wheel_length/2} 0" rpy="-${pi/2} 0 0"/>
-		<axis xyz="0 0 1"/>
-	</joint>
-	<link name="front_left_wheel_link">
-		<visual>
-			<geometry> <!-- the weheels are 60mm diameter, 25mm thick. -->
-				<cylinder radius="${wheel_radius}" length="${wheel_length}"/>
-			</geometry>
-			<material name="black"/>
-		</visual>
-		<collision>
-            <origin xyz="0 0 0" rpy="0 0 0"/>
-            <geometry>
-                <cylinder length="${wheel_length}" radius="${wheel_radius}" />
-            </geometry>
-        </collision>
-        <xacro:inertial_cylinder mass="1.0" length="${wheel_length}" radius="${wheel_radius}">
-            <origin xyz="0 0 0" rpy="0 0 0"/>
-        </xacro:inertial_cylinder>
-	</link>
+	<xacro:wheel_joint
+		name="front_left_wheel_joint"
+		parent="base_link"
+		child="front_left_wheel_link"
+		xyz="${chassis_length/4} ${chassis_length/2 + wheel_length/2} 0"
+		side="left">
+	</xacro:wheel_joint>
+	<xacro:wheel_link
+		name="front_left_wheel_link"
+		in_radius="${wheel_radius}"
+		in_length="${wheel_length}"
+		in_mass="${wheel_mass}">
+	</xacro:wheel_link>
 	<!-- front right wheel -->
-	<joint name="front_right_wheel_joint" type = "continuous">
-		<parent link="base_link"/>
-		<child link="front_right_wheel_link"/>
-		<origin xyz="${chassis_length/4} -${chassis_length/2 + wheel_length/2} 0" rpy="${pi/2} 0 0"/>
-		<axis xyz="0 0 -1"/>
-	</joint>
-	<link name="front_right_wheel_link">
-		<visual>
-			<geometry> <!-- the weheels are 60mm diameter, 25mm thick. -->
-				<cylinder length="${wheel_length}" radius="${wheel_radius}"/>
-			</geometry>
-			<material name="black"/>
-		</visual>
-		<collision>
-            <origin xyz="0 0 0" rpy="0 0 0"/>
-            <geometry>
-                <cylinder length="${wheel_length}" radius="${wheel_radius}" />
-            </geometry>
-        </collision>
-        <xacro:inertial_cylinder mass="1.0" length="${wheel_length}" radius="${wheel_radius}">
-            <!-- <origin xyz="${wheel_length/2} 0 0" rpy="0 ${pi/2} 0"/> -->
-            <origin xyz="0 0 0" rpy="0 0 0"/>
-        </xacro:inertial_cylinder>
-	</link>
+	<xacro:wheel_joint
+		name="front_right_wheel_joint"
+		parent="base_link"
+		child="front_right_wheel_link"
+		xyz="${chassis_length/4} -${chassis_length/2 + wheel_length/2} 0"
+		side="right">
+	</xacro:wheel_joint>
+	<xacro:wheel_link
+		name="front_right_wheel_link"
+		in_radius="${wheel_radius}"
+		in_length="${wheel_length}"
+		in_mass="${wheel_mass}">
+	</xacro:wheel_link>
 	<!-- rear left wheel -->
-	<joint name="rear_left_wheel_joint" type = "continuous">
-		<parent link="base_link"/>
-		<child link="rear_left_wheel_link"/>
-		<origin xyz="-${chassis_length/4} ${chassis_length/2 + wheel_length/2} 0" rpy="-${pi/2} 0 0"/>
-		<axis xyz="0 0 -1"/>
-	</joint>
-	<link name="rear_left_wheel_link">
-		<visual>
-			<geometry> <!-- the weheels are 60mm diameter, 25mm thick. -->
-				<cylinder length="${wheel_length}" radius="${wheel_radius}"/>
-			</geometry>
-			<material name="black"/>
-		</visual>
-		<collision>
-            <origin xyz="0 0 0" rpy="0 0 0"/>
-            <geometry>
-                <cylinder length="${wheel_length}" radius="${wheel_radius}" />
-            </geometry>
-        </collision>
-        <xacro:inertial_cylinder mass="1.0" length="${wheel_length}" radius="${wheel_radius}">
-            <origin xyz="0 0 0" rpy="0 0 0"/>
-        </xacro:inertial_cylinder>
-	</link>
+	<xacro:wheel_joint
+		name="rear_left_wheel_joint"
+		parent="base_link"
+		child="rear_left_wheel_link"
+		xyz="-${chassis_length/4} ${chassis_length/2 + wheel_length/2} 0"
+		side="left">
+	</xacro:wheel_joint>
+	<xacro:wheel_link
+		name="rear_left_wheel_link"
+		in_radius="${wheel_radius}"
+		in_length="${wheel_length}"
+		in_mass="${wheel_mass}">
+	</xacro:wheel_link>
 	<!-- rear right wheel -->
-	<joint name="rear_right_wheel_joint" type = "continuous">
-		<parent link="base_link"/>
-		<child link="rear_right_wheel_link"/>
-		<origin xyz="-${chassis_length/4} -${chassis_length/2 + wheel_length/2} 0" rpy="${pi/2} 0 0"/>
-		<axis xyz="0 0 -1"/>
-	</joint>
-	<link name="rear_right_wheel_link">
-		<visual>
-			<geometry> <!-- the weheels are 60mm diameter, 25mm thick. -->
-				<cylinder length="${wheel_length}" radius="${wheel_radius}" />
-			</geometry>
-			<material name="black"/>
-		</visual>
-		<collision>
-            <origin xyz="0 0 0" rpy="0 0 0"/>
-            <geometry>
-                <cylinder length="${wheel_length}" radius="${wheel_radius}" />
-            </geometry>
-        </collision>
-        <xacro:inertial_cylinder mass="1.0" length="${wheel_length}" radius="${wheel_radius}">
-            <origin xyz="0 0 0" rpy="0 0 0"/>
-        </xacro:inertial_cylinder>
-	</link>
+	<xacro:wheel_joint
+		name="rear_right_wheel_joint"
+		parent="base_link"
+		child="rear_right_wheel_link"
+		xyz="-${chassis_length/4} -${chassis_length/2 + wheel_length/2} 0"
+		side="right">
+	</xacro:wheel_joint>
+	<xacro:wheel_link
+		name="rear_right_wheel_link"
+		in_radius="${wheel_radius}"
+		in_length="${wheel_length}"
+		in_mass="${wheel_mass}">
+	</xacro:wheel_link>
 </robot>

Commit message: parameterised damping and friction on the wheels

File: description/robot.gazebo.xacro (robot description, xacro)
@@ -85,26 +85,4 @@
         </sensor>
     </gazebo>
-    <!--
-    <gazebo>
-	  <plugin name="skid_steer_drive_controller" filename="libgazebo_ros_skid_steer_drive.so">
-	    <updateRate>100.0</updateRate>
-	    <robotNamespace>/</robotNamespace>
-	    <leftFrontJoint>front_left_wheel_joint</leftFrontJoint>
-	    <rightFrontJoint>front_right_wheel_joint</rightFrontJoint>
-	    <leftRearJoint>rear_left_wheel_joint</leftRearJoint>
-	    <rightRearJoint>rear_right_wheel_joint</rightRearJoint>
-	    <wheelSeparation>${chassis_width}</wheelSeparation>
-	    <wheelDiameter>${wheel_radius *2}</wheelDiameter>
-	    <robotBaseFrame>base_link</robotBaseFrame>
-	    <wheelTorque>20</wheelTorque>
-	    <commandTopic>cmd_vel</commandTopic>
-	    <odometryTopic>odom</odometryTopic>
-	    <odometryFrame>odom</odometryFrame>
-	    <broadcastTF>true</broadcastTF>
-	    <covariance_x>0.001</covariance_x>
-	    <covariance_y>0.001</covariance_y>
-	    <covariance_yaw>0.01</covariance_yaw>
-	  </plugin>
-	</gazebo> -->
 	<gazebo>
         <plugin name='diff_drive' filename='libgazebo_ros_diff_drive.so'>

File: description/robot.include.xacro (robot description, xacro)
@@ -30,5 +30,5 @@
         </inertial>
     </xacro:macro>
-    <xacro:macro name="wheel_joint" params="name parent child xyz side">
+    <xacro:macro name="wheel_joint" params="name parent child xyz side damping friction">
       <joint name="${name}" type="continuous">
         <parent link="${parent}" />
@@ -42,5 +42,5 @@
             <axis xyz="0 0 -1"/>
         </xacro:if>
-        <dynamics damping="10.0" friction="10.0"/>
+        <dynamics damping="${damping}" friction="${friction}"/>
       </joint>
     </xacro:macro>

File: description/robot.wheels.xacro (robot description, xacro)
@@ -5,11 +5,12 @@
     <xacro:property name="wheel_radius" value="0.025" />
     <xacro:property name="wheel_mass" value="1.0"/>
+    <xacro:property name="wheel_damping" value="5.0"/>
+    <xacro:property name="wheel_friction" value="5.0"/>
 	<!-- front left wheel -->
 	<xacro:wheel_joint
 		name="front_left_wheel_joint"
-		parent="base_link"
-		child="front_left_wheel_link"
+		parent="base_link" child="front_left_wheel_link"
 		xyz="${chassis_length/4} ${chassis_length/2 + wheel_length/2} 0"
-		side="left">
+		side="left" damping="${wheel_damping}" friction="${wheel_friction}">
 	</xacro:wheel_joint>
 	<xacro:wheel_link
@@ -22,8 +23,7 @@
 	<xacro:wheel_joint
 		name="front_right_wheel_joint"
-		parent="base_link"
-		child="front_right_wheel_link"
+		parent="base_link" child="front_right_wheel_link"
 		xyz="${chassis_length/4} -${chassis_length/2 + wheel_length/2} 0"
-		side="right">
+		side="right" damping="${wheel_damping}" friction="${wheel_friction}">
 	</xacro:wheel_joint>
 	<xacro:wheel_link
@@ -36,8 +36,7 @@
 	<xacro:wheel_joint
 		name="rear_left_wheel_joint"
-		parent="base_link"
-		child="rear_left_wheel_link"
+		parent="base_link" child="rear_left_wheel_link"
 		xyz="-${chassis_length/4} ${chassis_length/2 + wheel_length/2} 0"
-		side="left">
+		side="left" damping="${wheel_damping}" friction="${wheel_friction}">
 	</xacro:wheel_joint>
 	<xacro:wheel_link
@@ -50,8 +49,7 @@
 	<xacro:wheel_joint
 		name="rear_right_wheel_joint"
-		parent="base_link"
-		child="rear_right_wheel_link"
+		parent="base_link" child="rear_right_wheel_link"
 		xyz="-${chassis_length/4} -${chassis_length/2 + wheel_length/2} 0"
-		side="right">
+		side="right" damping="${wheel_damping}" friction="${wheel_friction}">
 	</xacro:wheel_joint>
 	<xacro:wheel_link
