Commit message: switchable ros2 control hardware interfaces and diff drive controllers + bunch of urdf changes to make it simulate better. still needs work, cos it wheelies.

File: description/robot.camera.xacro (robot description, xacro)
@@ -1,9 +1,11 @@
 <?xml version="1.0"?>
 <robot xmlns:xacro="http://www.ros.org/wiki/xacro">
-    <xacro:property name="camera_height" value="0.15" />
-    <xacro:property name="camera_width" value="0.15" />
-    <xacro:property name="camera_length" value="0.06" />
-    <xacro:property name="lens_radius" value="0.04" />
-    <xacro:property name="lens_length" value="0.06" />
+    <xacro:property name="camera_height" value="0.05" />
+    <xacro:property name="camera_width" value="0.05" />
+    <xacro:property name="camera_length" value="0.03" />
+    <xacro:property name="camera_mass" value="0.1" />
+    <xacro:property name="lens_radius" value="0.01" />
+    <xacro:property name="lens_length" value="0.03" />
+    <xacro:property name="camera_weight" value="0.03" />
 	<!-- camera_joint describes where the camera is relative to the arm -->
     <!-- - Even though the camera isn't moving relative to the arm, it will probably be helpful to have its own link/frame rather than just adding more visuals to the arm -->
@@ -39,7 +41,17 @@
             </geometry>
         </collision>
-        <xacro:inertial_box mass="0.1" x="${camera_length *2}" y="${camera_width}" z="${camera_height}">
+        <xacro:inertial_box mass="${camera_mass}" x="${camera_length *2}" y="${camera_width}" z="${camera_height}">
             <origin xyz="0.0 0 0" rpy="0 0 0"/>
         </xacro:inertial_box>
     </link>
+    <!-- Due to a quirk of how cameras work, an extra joint/link is required to create an
+            "optical frame" for the sensor. That isn't the focus for this tutorial, but you can
+            look at https://www.ros.org/reps/rep-0103.html#suffix-frames for slightly more information. -->
+    <!-- First, create the link and joint for the optical frame -->
+    <joint name="camera_optical_joint" type="fixed">
+        <origin xyz="0 0 0" rpy="-1.571 0 -1.571" />
+        <parent link="camera_link" />
+        <child link="camera_link_optical" />
+    </joint>
+    <link name="camera_link_optical"></link>
 </robot>

File: description/robot.core.xacro (robot description, xacro)
@@ -1,41 +1,10 @@
 <?xml version="1.0"?>
-<robot xmlns:xacro="http://www.ros.org/wiki/xacro" name="robot">
+<robot xmlns:xacro="http://www.ros.org/wiki/xacro">
 	<xacro:include filename="robot.include.xacro" />
 	<!-- base link -->
 	<link name="base_link">
 	</link>
-	<!-- chassis
-	  setting length/width/height as properties so we can do maths ops with them.
-	-->
-	<!-- 300mm (x) 300mm (y) and 50mm (z) -->
-	<xacro:property name="chassis_length" value="0.3" />
-    <xacro:property name="chassis_width" value="0.3" />
-    <xacro:property name="chassis_height" value="0.05" />
-	<joint name="chassis_joint" type="fixed">
-		<parent link="base_link"/>
-		<child link="chassis_link"/>
-		<origin xyz="-${chassis_length/2} 0 0"/>
-	</joint>
-	<link name="chassis_link">
-		<visual>
-			<!-- position chassis origin 1/2 chassis lenght relative to the link. -->
-			<origin xyz = "${chassis_length/2} 0 ${chassis_height/2}"/>
-			<geometry>
-				<box size="${chassis_length} ${chassis_width} ${chassis_height}"/>
-			</geometry>
-			<material name="orange"/>
-		</visual>
-		<collision>
-            <origin xyz="${chassis_length/2} 0 ${chassis_height/2}" rpy="0 0 0"/>
-            <geometry>
-                <box size="${chassis_length} ${chassis_width} ${chassis_height}" />
-            </geometry>
-        </collision>
-        <xacro:inertial_box mass="0.1" x="${chassis_length}" y="${chassis_width}" z="${chassis_height}">
-            <origin xyz="${chassis_length/2} 0 ${chassis_height/2}" rpy="0 0 0"/>
-        </xacro:inertial_box>
-	</link>
+	<xacro:include filename="robot.chassis.xacro" />
 	<xacro:include filename="robot.wheels.xacro" />
 	<xacro:include filename="robot.camera.xacro" />
-	<xacro:include filename="robot.gazebo.xacro" />
 </robot>

File: description/robot.gazebo.xacro (robot description, xacro)
@@ -42,15 +42,5 @@
 		</plugin>
 	</gazebo>
-	<!-- Due to a quirk of how cameras work, an extra joint/link is required to create an
-            "optical frame" for the sensor. That isn't the focus for this tutorial, but you can
-            look at https://www.ros.org/reps/rep-0103.html#suffix-frames for slightly more information. -->
-    <!-- First, create the link and joint for the optical frame -->
-    <joint name="camera_optical_joint" type="fixed">
-        <origin xyz="0 0 0" rpy="-1.571 0 -1.571" />
-        <parent link="camera_link" />
-        <child link="camera_link_optical" />
-    </joint>
-    <link name="camera_link_optical"></link>
-     <!-- Add a gazebo tag for the ORIGINAL camera_link (but in the plugin we reference the optical frame so that ROS can orient things correctly) -->
+	<!-- Add a gazebo tag for the ORIGINAL camera_link (but in the plugin we reference the optical frame so that ROS can orient things correctly) -->
     <!-- Within the gazebo tag we have the sensor tag, and inside that there is (among other things) the camera tag with the camera parameters,
             and the plugin tag with some extra parameters the plugin needs. -->
@@ -85,26 +75,3 @@
         </sensor>
     </gazebo>
-	<gazebo>
-        <plugin name='diff_drive' filename='libgazebo_ros_diff_drive.so'>
-            <!-- Wheel Information -->
-            <num_wheel_pairs>2</num_wheel_pairs>
-            <left_joint>front_left_wheel_joint</left_joint>
-            <left_joint>rear_left_wheel_joint</left_joint>
-            <right_joint>front_right_wheel_joint</right_joint>
-            <right_joint>rear_right_wheel_joint</right_joint>
-            <wheel_separation>${chassis_width}</wheel_separation>
-            <wheel_separation>${chassis_width}</wheel_separation>
-            <wheel_diameter>${wheel_radius * 2}</wheel_diameter>
-            <wheel_diameter>${wheel_radius * 2}</wheel_diameter>
-            <!-- Limits -->
-            <max_wheel_torque>200</max_wheel_torque>
-            <max_wheel_acceleration>10.0</max_wheel_acceleration>
-            <!-- Output -->
-            <odometry_frame>odom</odometry_frame>
-            <robot_base_frame>base_link</robot_base_frame>
-            <publish_odom>true</publish_odom>
-            <publish_odom_tf>true</publish_odom_tf>
-            <publish_wheel_tf>true</publish_wheel_tf>
-        </plugin>
-    </gazebo>
 </robot>

File: description/robot.include.xacro (robot description, xacro)
@@ -30,5 +30,5 @@
         </inertial>
     </xacro:macro>
-    <xacro:macro name="wheel_joint" params="name parent child xyz side damping friction">
+    <xacro:macro name="wheel_joint" params="name parent child xyz side damping friction max_effort max_velocity">
       <joint name="${name}" type="continuous">
         <parent link="${parent}" />
@@ -36,11 +36,12 @@
         <xacro:if value="${side == 'left'}">
             <origin xyz="${xyz}" rpy="-${pi/2} 0 0"/>
-            <axis xyz="0 0 1"/>
+            <axis xyz="0 0 -1"/>
         </xacro:if>
         <xacro:if value="${side == 'right'}">
             <origin xyz="${xyz}" rpy="${pi/2} 0 0"/>
-            <axis xyz="0 0 -1"/>
+            <axis xyz="0 0 1"/>
         </xacro:if>
         <dynamics damping="${damping}" friction="${friction}"/>
+        <limit effort="${max_effort}" velocity="${max_velocity}"/>
       </joint>
     </xacro:macro>
@@ -61,7 +62,18 @@
             </collision>
             <xacro:inertial_cylinder mass="${in_mass}" length="${in_length}" radius="${in_radius}">
+                <!-- I think the origin is the centre of mass - middle of the cylinder -->
                 <origin xyz="0 0 0" rpy="0 0 0"/>
             </xacro:inertial_cylinder>
         </link>
+    </xacro:macro>
+    <xacro:macro name="ros2control_wheel" params="joint_name cmd_min cmd_max">
+        <joint name="${joint_name}">
+            <command_interface name="velocity">
+                <param name="min">${cmd_min}</param>
+                <param name="max">${cmd_max}</param>
+            </command_interface>
+            <state_interface name="velocity"/>
+            <state_interface name="position"/>
+        </joint>
     </xacro:macro>
     <!-- materials -->

File: description/robot.urdf.xacro (robot description, xacro)
@@ -1,4 +1,21 @@
 <?xml version="1.0"?>
 <robot xmlns:xacro="http://www.ros.org/wiki/xacro"  name="robot">
+     <xacro:arg name="use_ros2_control" default="true"/>
+    <!-- define the robot structure -->
     <xacro:include filename="robot.core.xacro" />
+    <!-- gazebo materials definitions and gazebo reporting joint states and camera feed from sim. -->
+    <xacro:include filename="robot.gazebo.xacro" />
+    <!-- gazebo represents and controls the robot via diff drive.  camera etc
+        comment out when using either gazebo or hardware ros2 control. -->
+    <!-- <xacro:include filename="robot.gazebo.control.xacro" /> -->
+    <!-- make a choice about ros control - hardware or simulation -->
+    <xacro:if value="$(arg use_ros2_control)">
+        <!-- USE ROS2 CONTROL is true -->
+        <xacro:include filename="robot.ros2.control.xacro" />
+    </xacro:if>
+    <xacro:unless value="$(arg use_ros2_control)">
+        <!-- USE ROS2 CONTROL is false -->
+        <xacro:include filename="robot.gazebo.roscontrol.xacro" />
+    </xacro:unless>
+    <!-- Should have chosen one by now -->
 </robot>

File: description/robot.wheels.xacro (robot description, xacro)
@@ -2,9 +2,11 @@
 <robot xmlns:xacro="http://www.ros.org/wiki/xacro">
 <!-- all the wheels -->
-	<xacro:property name="wheel_length" value="0.03" />
-    <xacro:property name="wheel_radius" value="0.025" />
-    <xacro:property name="wheel_mass" value="1.0"/>
-    <xacro:property name="wheel_damping" value="5.0"/>
-    <xacro:property name="wheel_friction" value="5.0"/>
+	<xacro:property name="wheel_length" value="0.025" />
+    <xacro:property name="wheel_radius" value="0.03" />
+    <xacro:property name="wheel_mass" value="0.027"/>
+    <xacro:property name="wheel_damping" value="1.0"/>
+    <xacro:property name="wheel_friction" value="1.0"/>
+    <xacro:property name="wheel_max_effort" value="0.5"/>
+    <xacro:property name="wheel_max_velocity" value="1.0"/>
 	<!-- front left wheel -->
 	<xacro:wheel_joint
@@ -12,5 +14,6 @@
 		parent="base_link" child="front_left_wheel_link"
 		xyz="${chassis_length/4} ${chassis_length/2 + wheel_length/2} 0"
-		side="left" damping="${wheel_damping}" friction="${wheel_friction}">
+		side="left" damping="${wheel_damping}" friction="${wheel_friction}"
+		max_effort="${wheel_max_effort}" max_velocity="${wheel_max_velocity}">
 	</xacro:wheel_joint>
 	<xacro:wheel_link
@@ -25,5 +28,6 @@
 		parent="base_link" child="front_right_wheel_link"
 		xyz="${chassis_length/4} -${chassis_length/2 + wheel_length/2} 0"
-		side="right" damping="${wheel_damping}" friction="${wheel_friction}">
+		side="right" damping="${wheel_damping}" friction="${wheel_friction}"
+		max_effort="${wheel_max_effort}" max_velocity="${wheel_max_velocity}">
 	</xacro:wheel_joint>
 	<xacro:wheel_link
@@ -38,5 +42,6 @@
 		parent="base_link" child="rear_left_wheel_link"
 		xyz="-${chassis_length/4} ${chassis_length/2 + wheel_length/2} 0"
-		side="left" damping="${wheel_damping}" friction="${wheel_friction}">
+		side="left" damping="${wheel_damping}" friction="${wheel_friction}"
+		max_effort="${wheel_max_effort}" max_velocity="${wheel_max_velocity}">
 	</xacro:wheel_joint>
 	<xacro:wheel_link
@@ -51,5 +56,6 @@
 		parent="base_link" child="rear_right_wheel_link"
 		xyz="-${chassis_length/4} -${chassis_length/2 + wheel_length/2} 0"
-		side="right" damping="${wheel_damping}" friction="${wheel_friction}">
+		side="right" damping="${wheel_damping}" friction="${wheel_friction}"
+		max_effort="${wheel_max_effort}" max_velocity="${wheel_max_velocity}">
 	</xacro:wheel_joint>
 	<xacro:wheel_link
